File: pcb/Pinky3.sch (KiCad schematic (older format))
At the start: 58 parts, among them J1 MJ-4PP-9, P1 i2c-pin, P2 i2c-pin, SW1 RESET_SW, SW10 SW_PUSH, SW11 SW_PUSH, SW12 SW_PUSH, SW13 SW_PUSH, SW14 SW_PUSH, SW15 SW_PUSH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

Commit message: - add images - add logo - change thumb keys footprints to choc only
Parts:
- J1: symbol kbd:MJ-4PP-9 -> Pinky3-rescue:MJ-4PP-9-kbd
- SW1, SW10, SW11, SW12, SW13, SW15, SW16, SW17, SW19, SW2, SW20, SW21, SW23, SW24, SW25, SW3, SW4, SW5, SW6, SW7, SW8, SW9: symbol kbd:SW_PUSH -> Pinky3-rescue:SW_PUSH-kbd
- SW14, SW18, SW22, SW26: footprint kbd:CherryMX_KailhLowProfile_Hotswap -> kbd:Choc_Hotswap; symbol kbd:SW_PUSH -> Pinky3-rescue:SW_PUSH-kbd
- U1: symbol kbd:ProMicro -> Pinky3-rescue:ProMicro-kbd
Changed lines of the file:
@@
 EESchema Schematic File Version 4
-LIBS:Pinky-cache
+LIBS:Pinky3-cache
 EELAYER 26 0
 EELAYER END
@@
 $EndDescr
 $Comp
-L kbd:ProMicro U1
+L Pinky3-rescue:ProMicro-kbd U1
 U 1 1 5BC2FDFC
 P 1905 2195
@@
 	3055 1745 3055 1395
 $Comp
-L kbd:SW_PUSH SW5
+L Pinky3-rescue:SW_PUSH-kbd SW5
 U 1 1 5BC302DC
 P 5840 3570
@@
 reset
 $Comp
-L kbd:SW_PUSH SW1
+L Pinky3-rescue:SW_PUSH-kbd SW1
 U 1 1 5BC2BB1A
 P 1975 4845
@@
 data
 $Comp
-L kbd:MJ-4PP-9 J1
+L Pinky3-rescue:MJ-4PP-9-kbd J1
 U 1 1 5BCC34EB
 P 1655 3595
@@
 NoConn ~ 2605 2545
 $Comp
-L kbd:SW_PUSH SW3
+L Pinky3-rescue:SW_PUSH-kbd SW3
 U 1 1 5BD6F90B
 P 4920 4230
@@
 $EndComp
 $Comp
-L kbd:SW_PUSH SW4
+L Pinky3-rescue:SW_PUSH-kbd SW4
 U 1 1 5BD708BE
 P 4920 4910
@@
 $EndComp
 $Comp
-L kbd:SW_PUSH SW6
+L Pinky3-rescue:SW_PUSH-kbd SW6
 U 1 1 5BD70F56
 P 5840 4230
@@
 $EndComp
 $Comp
-L kbd:SW_PUSH SW7
+L Pinky3-rescue:SW_PUSH-kbd SW7
 U 1 1 5BD71F0E
 P 5840 4910
@@
 $EndComp
 $Comp
-L kbd:SW_PUSH SW2
+L Pinky3-rescue:SW_PUSH-kbd SW2
 U 1 1 5BC302D5
 P 4920 3570
@@
 $EndComp
 $Comp
-L kbd:SW_PUSH SW8
+L Pinky3-rescue:SW_PUSH-kbd SW8
 U 1 1 5BDBCD8D
 P 6730 3570
@@
 $EndComp
 $Comp
-L kbd:SW_PUSH SW11
+L Pinky3-rescue:SW_PUSH-kbd SW11
 U 1 1 5BDBD8D0
 P 7605 3570
@@
 $EndComp
 $Comp
-L kbd:SW_PUSH SW9
+L Pinky3-rescue:SW_PUSH-kbd SW9
 U 1 1 5BDBDE28
 P 6730 4230
@@
 $EndComp
 $Comp
-L kbd:SW_PUSH SW12
+L Pinky3-rescue:SW_PUSH-kbd SW12
 U 1 1 5BDBE29C
 P 7605 4230
@@
 $EndComp
 $Comp
-L kbd:SW_PUSH SW10
+L Pinky3-rescue:SW_PUSH-kbd SW10
 U 1 1 5BDBE802
 P 6730 4910
@@
 $EndComp
 $Comp
-L kbd:SW_PUSH SW13
+L Pinky3-rescue:SW_PUSH-kbd SW13
 U 1 1 5BDBECBA
 P 7605 4910
@@
 $EndComp
 $Comp
-L kbd:SW_PUSH SW14
+L Pinky3-rescue:SW_PUSH-kbd SW14
 U 1 1 5BDBF6B1
 P 7605 5570
 F 0 "SW14" H 7605 5825 50  0000 C CNN
 F 1 "SW_PUSH" H 7605 5734 50  0000 C CNN
-F 2 "kbd:CherryMX_KailhLowProfile_Hotswap" H 7605 5570 50  0001 C CNN
+F 2 "kbd:Choc_Hotswap" H 7605 5570 50  0001 C CNN
 F 3 "" H 7605 5570 50  0000 C CNN
 	1    7605 5570
@@
 $EndComp
 $Comp
-L kbd:SW_PUSH SW15
+L Pinky3-rescue:SW_PUSH-kbd SW15
 U 1 1 5BDC050F
 P 8460 3570
@@
 $EndComp
 $Comp
-L kbd:SW_PUSH SW16
+L Pinky3-rescue:SW_PUSH-kbd SW16
 U 1 1 5BDC09AE
 P 8460 4230
@@
 $EndComp
 $Comp
-L kbd:SW_PUSH SW17
+L Pinky3-rescue:SW_PUSH-kbd SW17
 U 1 1 5BDC0E41
 P 8460 4910
@@
 $EndComp
 $Comp
-L kbd:SW_PUSH SW18
+L Pinky3-rescue:SW_PUSH-kbd SW18
 U 1 1 5BDC1338
 P 8460 5570
 F 0 "SW18" H 8460 5825 50  0000 C CNN
 F 1 "SW_PUSH" H 8460 5734 50  0000 C CNN
-F 2 "kbd:CherryMX_KailhLowProfile_Hotswap" H 8460 5570 50  0001 C CNN
+F 2 "kbd:Choc_Hotswap" H 8460 5570 50  0001 C CNN
 F 3 "" H 8460 5570 50  0000 C CNN
 	1    8460 5570
@@
 $EndComp
 $Comp
-L kbd:SW_PUSH SW19
+L Pinky3-rescue:SW_PUSH-kbd SW19
 U 1 1 5BDC2CE9
 P 9300 3570
@@
 $EndComp
 $Comp
-L kbd:SW_PUSH SW20
+L Pinky3-rescue:SW_PUSH-kbd SW20
 U 1 1 5BDC2CF0
 P 9300 4230
@@
 $EndComp
 $Comp
-L kbd:SW_PUSH SW21
+L Pinky3-rescue:SW_PUSH-kbd SW21
 U 1 1 5BDC2CF7
 P 9300 4910
@@
 $EndComp
 $Comp
-L kbd:SW_PUSH SW22
+L Pinky3-rescue:SW_PUSH-kbd SW22
 U 1 1 5BDC2CFE
 P 9300 5570
 F 0 "SW22" H 9300 5825 50  0000 C CNN
 F 1 "SW_PUSH" H 9300 5734 50  0000 C CNN
-F 2 "kbd:CherryMX_KailhLowProfile_Hotswap" H 9300 5570 50  0001 C CNN
+F 2 "kbd:Choc_Hotswap" H 9300 5570 50  0001 C CNN
 F 3 "" H 9300 5570 50  0000 C CNN
 	1    9300 5570
@@
 	4335 5870 7905 5870
 $Comp
-L kbd:SW_PUSH SW23
+L Pinky3-rescue:SW_PUSH-kbd SW23
 U 1 1 5BF7CE09
 P 10185 3570
@@
 $EndComp
 $Comp
-L kbd:SW_PUSH SW24
+L Pinky3-rescue:SW_PUSH-kbd SW24
 U 1 1 5BF7CE10
 P 10185 4230
@@
 $EndComp
 $Comp
-L kbd:SW_PUSH SW25
+L Pinky3-rescue:SW_PUSH-kbd SW25
 U 1 1 5BF7CE17
 P 10185 4910
@@
 $EndComp
 $Comp
-L kbd:SW_PUSH SW26
+L Pinky3-rescue:SW_PUSH-kbd SW26
 U 1 1 5BF7CE1E
 P 10185 5570
 F 0 "SW26" H 10185 5825 50  0000 C CNN
 F 1 "SW_PUSH" H 10185 5734 50  0000 C CNN
-F 2 "kbd:CherryMX_KailhLowProfile_Hotswap" H 10185 5570 50  0001 C CNN
+F 2 "kbd:Choc_Hotswap" H 10185 5570 50  0001 C CNN
 F 3 "" H 10185 5570 50  0000 C CNN
 	1    10185 5570
