File: top-plate/Pinky3-top-plate.kicad_pcb (KiCad board)
At the start: 2 copper layers, 135.7 x 86.9 mm, 9 parts

Commit message: - add images - add logo - change thumb keys footprints to choc only
Parts:
- added G***: LOGO, lib:pinky3, B.Cu at (107.5, 112.2)
- added G***: LOGO, lib:pinky3, F.Cu at (107.5, 112.2)
Other:
- outline, holes or cut-outs redrawn
- board text removed: "rev. 0.3 @tamanishi"
